File: ql-flex.kicad_sch (KiCad schematic)
At the start: 15 parts, among them J1 QL_SLOT_DIN41612_FEMALE-90deg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, J2 QL_SLOT_DIN41612_MALE_90degre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, U1 HM628512BLFP-7, U2 GAL16V8B-25QP, U3 LM1117-5.0

Commit message: Update schematic title block with new project name and copyright
Other:
- company: (C) 2022 Alvaro Alea Fdz -> (C) 2026 Arley Silveira + (C) Alvaro Alea
- title: External Expansion 512Kb memory for Sinclair QL -> QL Flex Memory Expansion
Changed lines of the file:
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@@
 	(paper "A4")
 	(title_block
-		(title "External Expansion 512Kb memory for Sinclair QL")
-		(date "2024-11-22")
+		(title "QL Flex Memory Expansion")
+		(date "2026-08-07")
 		(rev "3")
-		(company "(C) 2022 Alvaro Alea Fdz")
+		(company "(C) 2026 Arley Silveira + (C) Alvaro Alea")
 		(comment 1 "https://ohwr.org/cern_ohl_s_v2.txt")
 		(comment 2 "CERN Open Hardware Licence Version 2 - Strongly Reciprocal")
